File: Hardware_Files/Project/IMU.kicad_sch (KiCad schematic)
At the start: 14 parts

Commit message: Repo Update
Parts:
- removed U?: BMI088, Footprint:PQFN50P450X300X100-16N, symbol BMI088:BMI088
- added U4: BMI088, Footprint:PQFN50P450X300X100-16N, symbol BMI088:BMI088
- C10, C11, C12, C13, C6, C7, C8, C9: renamed from C?; footprint (none) -> Capacitor_SMD:C_0201_0603Metric_Pad0.64x0.40mm_HandSolder
- R15, R16, R17, R18: renamed from R?; footprint (none) -> Resistor_SMD:R_0201_0603Metric_Pad0.64x0.40mm_HandSolder
- gave numbers to parts that had none: 1
Connections:
- net ACCL2_INT1: now also U4.16 (INT1)
- net ACCL2_INT2: now also U4.1 (INT2)
- net GND: now also U4.4 (GNDA), U4.6 (GNDIO)
- net GYRO2_INT1: now also U4.12 (INT3)
- net GYRO2_INT2: now also U4.13 (INT4)
- net I2C2_SCL: now also U4.8 (SCL/SCK)
- net I2C2_SDA: now also U4.9 (SDA/SDI)
- net VCC renamed +3V3
- net +3V3: now also U4.10 (SDO2), U4.11 (VDDIO), U4.15 (SDO1), U4.3 (VDD), U4.7 (PS)
