File: Hardware_Files/Project/PHY.kicad_sch (KiCad schematic)
At the start: 23 parts, among them J1 HR911105A, U1 LAN8720A-CP, Y1 ASCO-50.000MHZ-EK-T3

Commit message: Repo Update
Parts:
- added R23: 12.1K, Resistor_SMD:R_0201_0603Metric_Pad0.64x0.40mm_HandSolder, symbol Device:R_Small
- C1, C2, C3, C4, C5: footprint (none) -> Capacitor_SMD:C_0201_0603Metric_Pad0.64x0.40mm_HandSolder
- L1: footprint (none) -> Inductor_SMD:L_0402_1005Metric_Pad0.77x0.64mm_HandSolder
- R1, R10, R11, R12, R13, R14, R2, R3, R4, R5, R6, R7, R8, R9: footprint (none) -> Resistor_SMD:R_0201_0603Metric_Pad0.64x0.40mm_HandSolder
Connections:
- net GND: now also R23.2
- net RBIAS: no longer names the net of U1.24 (RBIAS)
- net RBIAS: now also R23.1
