File: Hardware_Files/Project/Project.kicad_sch (KiCad schematic)
At the start: 2 parts

Commit message: Repo Update
Parts:
- added C14, C15, C18, C20, C21: 104, Capacitor_SMD:C_0201_0603Metric_Pad0.64x0.40mm_HandSolder, symbol Device:C_Small
- added C16, C17: 2.2uF, Capacitor_SMD:C_0201_0603Metric_Pad0.64x0.40mm_HandSolder, symbol Device:C_Small
- added C19, C22: 106, Capacitor_SMD:C_0201_0603Metric_Pad0.64x0.40mm_HandSolder, symbol Device:C_Polarized_Small
- added C23: C_Polarized, Capacitor_SMD:CP_Elec_4x4.5, symbol Device:C_Polarized
- added H1, H2, H3, H4: MountingHole, MountingHole:MountingHole_2.2mm_M2_Pad_Via, symbol Mechanical:MountingHole
- added J2: Conn_01x10, Connector_PinHeader_1.00mm:PinHeader_1x10_P1.00mm_Vertical_SMD_Pin1Right, symbol Connector_Generic:Conn_01x10
- added J3, J4: Conn_01x06, Connector_PinHeader_1.00mm:PinHeader_1x06_P1.00mm_Vertical_SMD_Pin1Left, symbol Connector_Generic:Conn_01x06
- added J5: Conn_01x07, Connector_PinHeader_1.00mm:PinHeader_1x07_P1.00mm_Vertical_SMD_Pin1Left, symbol Connector_Generic:Conn_01x07
- added J6: S2B-PH-SM4-TB(LF)(SN), Footprint:JST_S2B-PH-SM4-TB(LF)(SN), symbol S2B-PH-SM4-TB_LF__SN_:S2B-PH-SM4-TB(LF)(SN)
- added R19, R22: 10K, Resistor_SMD:R_0201_0603Metric_Pad0.64x0.40mm_HandSolder, symbol Device:R_Small
- added R20, R21: 0R, Resistor_SMD:R_0201_0603Metric_Pad0.64x0.40mm_HandSolder, symbol Device:R_Small
- added U5: MAX7375AXR365, Package_TO_SOT_SMD:SOT-323_SC-70, symbol Oscillator:MAX7375AXR365
- added U6: AMS1117-3.3, Package_TO_SOT_SMD:SOT-223-3_TabPin2, symbol Regulator_Linear:AMS1117-3.3
- added X1: SG-3030CM, Oscillator:Oscillator_SMD_SeikoEpson_SG3030CM, symbol Oscillator:SG-3030CM
- BT1: renamed from BT?; footprint (none) -> Battery:BatteryHolder_Keystone_3000_1x12mm
- gave numbers to parts that had none: 1
Connections:
- net ACCL1_IN1: now also U2.35 (PB0), J3.3 (Pin_3)
- net ACCL1_INT2: now also U2.36 (PB1), J3.4 (Pin_4)
- net ETH_CRS_DV: now also J2.10 (Pin_10)
- net ETH_MDC: now also J2.8 (Pin_8)
- net ETH_MDIO: now also U2.24 (PA1), J2.9 (Pin_9); no longer U2.25 (PA2)
- net ETH_REF_CLK: now also U2.23 (PA0), J2.5 (Pin_5); no longer U2.24 (PA1)
- net ETH_RX_D0: now also J2.6 (Pin_6)
- net ETH_RX_D1: now also J2.7 (Pin_7)
- net ETH_TX_D0: now also J2.3 (Pin_3)
- net ETH_TX_D1: now also J2.4 (Pin_4)
- net ETH_TX_EN: now also J2.2 (Pin_2)
- net GND: now also C14.2, C15.2, C16.2, C17.2, C18.2, C19.2, C20.2, C21.2, C22.2, C23.2, J5.7 (Pin_7), J6.2, R19.2, R22.2, U5.3 (GND), U6.1 (GND), X1.2 (GND)
- net GYRO1_INT1: now also U2.17 (PC2), J3.5 (Pin_5)
- net GYRO1_INT2: now also U2.89 (PB3), J3.6 (Pin_6)
- net I2C1_SCL: now also U2.92 (PB6), J3.1 (Pin_1)
- net I2C1_SDA: now also U2.93 (PB7), J3.2 (Pin_2)
- net OSC_IN: now reaches U2.12 (PH0)
- net OSC_IN: now also U5.2 (CLOCK)
- net at U2.14 (NRST): now also C15.1
- net VREF+: now reaches U2.21 (VREF+)
- net VREF+: now also R21.1
- net at U2.37 (PB2): now also R22.1
- net at U2.49 (VCAP_1): now also C17.1
- net I2C3_SDA: now reaches U2.66 (PC9)
- net I2C3_SDA: now also J4.2 (Pin_2)
- net I2C3_SCL: now reaches U2.67 (PA8)
- net I2C3_SCL: now also J4.1 (Pin_1)
- net UART_TX: now reaches U2.68 (PA9)
- net UART_TX: now also J5.5 (Pin_5)
- net UART_RX: now reaches U2.69 (PA10)
- net UART_RX: now also J5.6 (Pin_6)
- net SWDIO: now reaches U2.72 (PA13)
- net SWDIO: now also J5.3 (Pin_3)
- net at U2.73 (VCAP_2): now also C16.1
- net SWCLK: now reaches U2.76 (PA14)
- net SWCLK: now also J5.4 (Pin_4)
- net OSC32_IN: now reaches U2.8 (PC14)
- net OSC32_IN: now also X1.3 (OUT)
- net ACCL2_IN1: now reaches U2.90 (PB4)
- net ACCL2_IN1: now also J4.3 (Pin_3)
- net ACCL2_INT2: now reaches U2.91 (PB5)
- net ACCL2_INT2: now also J4.4 (Pin_4)
- net at U2.94 (BOOT0): now also R19.1
- net GYRO2_INT1: now reaches U2.95 (PB8)
- net GYRO2_INT1: now also J4.5 (Pin_5)
- net GYRO2_INT2: now reaches U2.96 (PB9)
- net GYRO2_INT2: now also J4.6 (Pin_6)
- net VCC renamed +3V3
- net +3V3: now also C14.1, C21.1, C22.1, J5.1 (Pin_1), R20.1, U5.1 (V+), U6.2 (VO), X1.1 (VIO), X1.4 (Vcc)
- new net: J6.S1 (SHIELD), J6.S2 (SHIELD)
- new net +5V: C19.1, C20.1, C23.1, J5.2 (Pin_2), J6.1, U6.3 (VI)
- new net VDDA: C18.1, R20.2, R21.2
- new net nNRST: J2.1 (Pin_1), U2.25 (PA2)
- no-connect marks 0 -> 54
